Commit message: update

File: curobo/content/assets/robot/x7s_mobile/x7s_mobile.urdf (robot description, URDF)
Before this commit: robot X7S, 29 links, 28 joints
Joints:
- joint dummy_base_prismatic_x_joint: limit lower=-50 upper=50 effort=100 velocity=1000 -> lower=-5 upper=5 effort=100 velocity=1000
- joint dummy_base_prismatic_y_joint: limit lower=-50 upper=50 effort=100 velocity=1000 -> lower=-5 upper=5 effort=100 velocity=1000
- joint dummy_base_revolute_z_joint: limit lower=-3.14159 upper=3.14159 effort=100 velocity=1000 -> lower=-3.141593 upper=3.141593 effort=100 velocity=1000
- joint joint10: limit lower=-10 upper=10 effort=100 velocity=1000 -> lower=-3.141593 upper=3.141593 effort=100 velocity=1000
- joint joint11: limit lower=-10 upper=10 effort=100 velocity=100 -> lower=-3.141593 upper=3.141593 effort=100 velocity=100
- joint joint14: limit lower=-10 upper=10 effort=100 velocity=1000 -> lower=-3.141593 upper=3.141593 effort=100 velocity=1000
- joint joint15: limit lower=-10 upper=10 effort=100 velocity=1000 -> lower=-3.141593 upper=3.141593 effort=100 velocity=1000
- joint joint16: limit lower=-10 upper=10 effort=100 velocity=1000 -> lower=-3.141593 upper=3.141593 effort=100 velocity=1000
- joint joint17: limit lower=-10 upper=10 effort=100 velocity=1000 -> lower=-3.141593 upper=3.141593 effort=100 velocity=1000
- joint joint18: limit lower=-10 upper=10 effort=100 velocity=1000 -> lower=-3.141593 upper=3.141593 effort=100 velocity=1000
- joint joint19: limit lower=-10 upper=10 effort=100 velocity=1000 -> lower=-3.141593 upper=3.141593 effort=100 velocity=1000
- joint joint2: limit lower=-10 upper=10 effort=100 velocity=1000 -> lower=-3.141593 upper=3.141593 effort=100 velocity=1000
- joint joint20: limit lower=-10 upper=10 effort=100 velocity=1000 -> lower=-3.141593 upper=3.141593 effort=100 velocity=1000
- joint joint3: limit lower=-10 upper=10 effort=100 velocity=1000 -> lower=-3.141593 upper=3.141593 effort=100 velocity=1000
- joint joint4: limit lower=-10 upper=10 effort=100 velocity=1000 -> lower=-3.141593 upper=3.141593 effort=100 velocity=1000
- joint joint5: limit lower=-10 upper=10 effort=100 velocity=1000 -> lower=-3.141593 upper=3.141593 effort=100 velocity=1000
- joint joint6: limit lower=-10 upper=10 effort=100 velocity=1000 -> lower=-3.141593 upper=3.141593 effort=100 velocity=1000
- joint joint7: limit lower=-10 upper=10 effort=100 velocity=1000 -> lower=-3.141593 upper=3.141593 effort=100 velocity=1000
- joint joint8: limit lower=-10 upper=10 effort=100 velocity=1000 -> lower=-3.141593 upper=3.141593 effort=100 velocity=1000
- joint joint9: limit lower=-10 upper=10 effort=100 velocity=1000 -> lower=-3.141593 upper=3.141593 effort=100 velocity=1000

File: curobo/content/assets/robot/x7s_mobile/x7s_mobile_fix.urdf (robot description, URDF)
Before this commit: robot X7S, 29 links, 28 joints
Joints:
- joint joint10: limit lower=-10 upper=10 effort=100 velocity=1000 -> lower=-3.141593 upper=3.141593 effort=100 velocity=1000
- joint joint11: limit lower=-10 upper=10 effort=100 velocity=100 -> lower=-3.141593 upper=3.141593 effort=100 velocity=100
- joint joint14: limit lower=-10 upper=10 effort=100 velocity=1000 -> lower=-3.141593 upper=3.141593 effort=100 velocity=1000
- joint joint15: limit lower=-10 upper=10 effort=100 velocity=1000 -> lower=-3.141593 upper=3.141593 effort=100 velocity=1000
- joint joint16: limit lower=-10 upper=10 effort=100 velocity=1000 -> lower=-3.141593 upper=3.141593 effort=100 velocity=1000
- joint joint17: limit lower=-10 upper=10 effort=100 velocity=1000 -> lower=-3.141593 upper=3.141593 effort=100 velocity=1000
- joint joint18: limit lower=-10 upper=10 effort=100 velocity=1000 -> lower=-3.141593 upper=3.141593 effort=100 velocity=1000
- joint joint19: limit lower=-10 upper=10 effort=100 velocity=1000 -> lower=-3.141593 upper=3.141593 effort=100 velocity=1000
- joint joint2: limit lower=-10 upper=10 effort=100 velocity=1000 -> lower=-3.141593 upper=3.141593 effort=100 velocity=1000
- joint joint20: limit lower=-10 upper=10 effort=100 velocity=1000 -> lower=-3.141593 upper=3.141593 effort=100 velocity=1000
- joint joint3: limit lower=-10 upper=10 effort=100 velocity=1000 -> lower=-3.141593 upper=3.141593 effort=100 velocity=1000
- joint joint4: limit lower=-10 upper=10 effort=100 velocity=1000 -> lower=-3.141593 upper=3.141593 effort=100 velocity=1000
- joint joint5: limit lower=-10 upper=10 effort=100 velocity=1000 -> lower=-3.141593 upper=3.141593 effort=100 velocity=1000
- joint joint6: limit lower=-10 upper=10 effort=100 velocity=1000 -> lower=-3.141593 upper=3.141593 effort=100 velocity=1000
- joint joint7: limit lower=-10 upper=10 effort=100 velocity=1000 -> lower=-3.141593 upper=3.141593 effort=100 velocity=1000
- joint joint8: limit lower=-10 upper=10 effort=100 velocity=1000 -> lower=-3.141593 upper=3.141593 effort=100 velocity=1000
- joint joint9: limit lower=-10 upper=10 effort=100 velocity=1000 -> lower=-3.141593 upper=3.141593 effort=100 velocity=1000
