Commit message: g1 fixed hand

File: curobo/content/assets/robot/g1_simple/g1_fixed_hand.urdf (robot description, URDF)
Before this commit: robot g1_29dof_with_hand_rev_1_0, 37 links, 36 joints
Joints:
- joint waist_pitch_joint: limit lower=-0.1199999 upper=0.3199999 effort=50. velocity=37.0000001 -> lower=-1.5 upper=1.5 effort=50 velocity=37.0
- joint waist_roll_joint: limit lower=-0.1199999 upper=0.1199999 effort=50. velocity=37.0000001 -> lower=-1.0 upper=1.0 effort=50 velocity=37.0

File: curobo/content/assets/robot/g1_simple/g1_fixed_hand_mobile.urdf (robot description, URDF)
Before this commit: robot g1_29dof_with_hand_rev_1_0, 37 links, 36 joints
Links:
- added link base_link_h, mass 0.0001
- added link base_link_x, mass 0.0001
- added link base_link_y, mass 0.0001
- added link base_link_z, mass 0.0001
- added link g1_mobile
Joints:
- added joint base_fixed: type fixed, parent base_link_z, child g1_29dof_with_hand_rev_1_0, origin xyz=0 0 0.0 rpy=0 0 0.0, axis 0 0 0
- added joint base_h: type prismatic, parent base_link_y, child base_link_h, origin xyz=0 0 0.0 rpy=0 0 0.0, axis 0 0 1, limit lower=-1 upper=1 effort=87 velocity=1.50
- added joint base_x: type prismatic, parent g1_mobile, child base_link_x, origin xyz=0 0 0.0 rpy=0 0 0.0, axis 1 0 0, limit lower=-2 upper=2 effort=87 velocity=1.0
- added joint base_y: type prismatic, parent base_link_x, child base_link_y, origin xyz=0 0 0.0 rpy=0 0 0.0, axis 0 1 0, limit lower=-2 upper=2 effort=87 velocity=1.0
- added joint base_z: type revolute, parent base_link_h, child base_link_z, origin xyz=0 0 0.0 rpy=0 0 0.0, axis 0 0 1, limit lower=-180 upper=180 effort=87 velocity=1.50
- joint waist_pitch_joint: limit lower=-0.1199999 upper=0.3199999 effort=50. velocity=37.0000001 -> lower=-1.5 upper=1.5 effort=50 velocity=37.0
- joint waist_roll_joint: limit lower=-0.1199999 upper=0.1199999 effort=50. velocity=37.0000001 -> lower=-1.0 upper=1.0 effort=50 velocity=37.0
- joint waist_yaw_joint: limit lower=-1.618 upper=1.618 effort=88. velocity=32.0000004 -> lower=-2.618 upper=2.618 effort=88. velocity=32.0000004

File: curobo/content/assets/robot/vega_1p_sharpa/vega_1p_sharpa_fix.urdf (robot description, URDF)
Before this commit: robot vega_1p_sharpa, 107 links, 106 joints
Joints:
- joint torso_j1: limit lower=0. upper=0.785 effort=700. velocity=0.8999999 -> lower=0. upper=1.5699999 effort=700. velocity=0.8999999
