Commit message: update

File: curobo/content/assets/robot/dual_franka_description/urdf/dual_franka.urdf (robot description, URDF)
Before this commit: robot dual_franka, 25 links, 24 joints
Joints:
- joint base_to_L_panda_link0: origin xyz=0 0.9 0 rpy=0 0 -1.57079632679 -> xyz=0 0.7 0 rpy=0 0 -1.57079632679
- joint base_to_R_panda_link0: origin xyz=0 -0.9 0 rpy=0 0 1.57079632679 -> xyz=0 -0.7 0 rpy=0 0 1.57079632679

Commit message: vega1p sharpa

File: curobo/content/assets/robot/dual_franka_description/urdf/dual_franka.urdf (robot description, URDF)
Before this commit: robot dual_franka, 25 links, 24 joints
Joints:
- joint base_to_L_panda_link0: origin xyz=0 0.7 0 rpy=0 0 -1.57079632679 -> xyz=0 0.5 0 rpy=0 0 -1.57079632679
- joint base_to_R_panda_link0: origin xyz=0 -0.7 0 rpy=0 0 1.57079632679 -> xyz=0 -0.5 0 rpy=0 0 1.57079632679

Commit message: add flag and adjust dual franka

File: curobo/content/assets/robot/dual_franka_description/urdf/dual_franka.urdf (robot description, URDF)
Before this commit: robot dual_franka, 25 links, 24 joints
Joints:
- joint base_to_L_panda_link0: origin xyz=0 0.5 0 rpy=0 0 -1.57079632679 -> xyz=0 0.7 0 rpy=0 0 -1.57079632679
- joint base_to_R_panda_link0: origin xyz=0 -0.5 0 rpy=0 0 1.57079632679 -> xyz=0 -0.7 0 rpy=0 0 1.57079632679
