Commit message: Modified URDF to limit the waist joint movement

File: curobo/content/assets/robot/g1_dex1_head/g1_dex1_head.urdf (robot description, URDF)
Before this commit: robot g1_dex1_head, 58 links, 57 joints
Joints:
- joint waist_pitch_joint: limit lower=-1.5 upper=1.5 effort=50 velocity=37.0 -> lower=-0.1 upper=0.1 effort=50 velocity=37.0
- joint waist_roll_joint: limit lower=-1.0 upper=1.0 effort=50 velocity=37.0 -> lower=-0.1 upper=0.1 effort=50 velocity=37.0
- joint waist_yaw_joint: limit lower=-1.618 upper=1.618 effort=88. velocity=32.0000004 -> lower=-0.5 upper=0.5 effort=88. velocity=32.0000004

File: curobo/content/assets/robot/g1_dex1_head/g1_dex1_head_mobile.urdf (robot description, URDF)
Before this commit: robot g1_dex1_head_mobile, 63 links, 62 joints
Joints:
- joint waist_pitch_joint: limit lower=-1.5 upper=1.5 effort=50 velocity=37.0 -> lower=-0.1 upper=0.1 effort=50 velocity=37.0
- joint waist_roll_joint: limit lower=-1.0 upper=1.0 effort=50 velocity=37.0 -> lower=-0.1 upper=0.1 effort=50 velocity=37.0
- joint waist_yaw_joint: limit lower=-2.618 upper=2.618 effort=88. velocity=32.0000004 -> lower=-0.5 upper=0.5 effort=88. velocity=32.0000004
