Commit message: lmb(dex1-head): waist limits use the large range (yaw 2.618, roll/pitch 0.52) like g1_dex1.urdf and the USD
The URDF narrowed them to 0.5 / 0.1 / 0.1, which also limited the cuRobo free-base model (plus the 0.2 rad position_limit_clip).

Co-Authored-By: Claude Sonnet 5.5 <noreply@anthropic.com>

File: curobo/content/assets/robot/g1_dex1_head/g1_dex1_head.urdf (robot description, URDF)
Before this commit: robot g1_dex1_head, 58 links, 57 joints
Joints:
- joint waist_pitch_joint: limit lower=-0.1 upper=0.1 effort=50 velocity=37.0 -> lower=-0.52 upper=0.52 effort=50 velocity=37.0
- joint waist_roll_joint: limit lower=-0.1 upper=0.1 effort=50 velocity=37.0 -> lower=-0.52 upper=0.52 effort=50 velocity=37.0
- joint waist_yaw_joint: limit lower=-0.5 upper=0.5 effort=88. velocity=32.0000004 -> lower=-2.618 upper=2.618 effort=88. velocity=32.0000004

File: curobo/content/assets/robot/g1_dex1_head/g1_dex1_head_mobile.urdf (robot description, URDF)
Before this commit: robot g1_dex1_head_mobile, 63 links, 62 joints
Joints:
- joint waist_pitch_joint: limit lower=-0.1 upper=0.1 effort=50 velocity=37.0 -> lower=-0.52 upper=0.52 effort=50 velocity=37.0
- joint waist_roll_joint: limit lower=-0.1 upper=0.1 effort=50 velocity=37.0 -> lower=-0.52 upper=0.52 effort=50 velocity=37.0
- joint waist_yaw_joint: limit lower=-0.5 upper=0.5 effort=88. velocity=32.0000004 -> lower=-2.618 upper=2.618 effort=88. velocity=32.0000004
