Commit message: add dual

File: curobo/content/assets/robot/dual_arx_x5_description/urdf/dual_arx_x5.urdf (robot description, URDF)
Before this commit: robot dual_arx_x5, 19 links, 18 joints
Links:
- link L_base_link: geometry collision mesh filename=package://arx_x5_description/meshes/base_link.STL; visual mesh filename=package://arx_x5_description/meshes/base_link.STL
- link L_link1: geometry collision mesh filename=package://arx_x5_description/meshes/link1.STL; visual mesh filename=package://arx_x5_description/meshes/link1.STL
- link L_link2: geometry collision mesh filename=package://arx_x5_description/meshes/link2.STL; visual mesh filename=package://arx_x5_description/meshes/link2.STL
- link L_link3: geometry collision mesh filename=package://arx_x5_description/meshes/link3.STL; visual mesh filename=package://arx_x5_description/meshes/link3.STL
- link L_link4: geometry collision mesh filename=package://arx_x5_description/meshes/link4.STL; visual mesh filename=package://arx_x5_description/meshes/link4.STL
- link L_link5: geometry collision mesh filename=package://arx_x5_description/meshes/link5.STL; visual mesh filename=package://arx_x5_description/meshes/link5.STL
- link L_link6: geometry collision mesh filename=package://arx_x5_description/meshes/link6.STL; visual mesh filename=package://arx_x5_description/meshes/link6.STL
- link L_link7: geometry collision mesh filename=package://arx_x5_description/meshes/link7.STL; visual mesh filename=package://arx_x5_description/meshes/link7.STL
- link L_link8: geometry collision mesh filename=package://arx_x5_description/meshes/link8.STL; visual mesh filename=package://arx_x5_description/meshes/link8.STL
- link R_base_link: geometry collision mesh filename=package://arx_x5_description/meshes/base_link.STL; visual mesh filename=package://arx_x5_description/meshes/base_link.STL
- link R_link1: geometry collision mesh filename=package://arx_x5_description/meshes/link1.STL; visual mesh filename=package://arx_x5_description/meshes/link1.STL
- link R_link2: geometry collision mesh filename=package://arx_x5_description/meshes/link2.STL; visual mesh filename=package://arx_x5_description/meshes/link2.STL
- link R_link3: geometry collision mesh filename=package://arx_x5_description/meshes/link3.STL; visual mesh filename=package://arx_x5_description/meshes/link3.STL
- link R_link4: geometry collision mesh filename=package://arx_x5_description/meshes/link4.STL; visual mesh filename=package://arx_x5_description/meshes/link4.STL
- link R_link5: geometry collision mesh filename=package://arx_x5_description/meshes/link5.STL; visual mesh filename=package://arx_x5_description/meshes/link5.STL
- link R_link6: geometry collision mesh filename=package://arx_x5_description/meshes/link6.STL; visual mesh filename=package://arx_x5_description/meshes/link6.STL
- link R_link7: geometry collision mesh filename=package://arx_x5_description/meshes/link7.STL; visual mesh filename=package://arx_x5_description/meshes/link7.STL
- link R_link8: geometry collision mesh filename=package://arx_x5_description/meshes/link8.STL; visual mesh filename=package://arx_x5_description/meshes/link8.STL
